File: igrow-101/$igrow-101.sch (KiCad schematic (older format))
At the start: 26 parts, among them P1 CONN_02X05, Q1 NPN, Q2 NPN, Q3 NPN, SW1 SW_PUSH, U1 NRF51822-MODULE, U2 SHT21, U3 TL972

Commit message: Post autorouting
Parts:
- PIEZO1: footprint Resistors_ThroughHole:Resistor_Vertical_RM5mm -> Resistors_SMD:R_0805_HandSoldering
Changed lines of the file:
@@
 F 0 "PIEZO1" H 4400 6450 40  0000 L CNN
 F 1 "PIEZO" H 4400 6350 40  0000 L CNN
-F 2 "Resistors_ThroughHole:Resistor_Vertical_RM5mm" H 4300 6400 60  0001 C CNN
+F 2 "Resistors_SMD:R_0805_HandSoldering" H 4300 6400 60  0001 C CNN
 F 3 "" H 4300 6400 60  0000 C CNN
 	1    4300 6400
