File: igrow-101/igrow-101.sch (KiCad schematic (older format))
At the start: 16 parts, among them P1 CONN_02X05, Q1 NPN, U1 NRF51822-MODULE, U2 SHT21

Commit message: Add simulation work and schematic/board WIP
Parts:
- added Q2, Q3: NPN, Housings_SOT-23_SOT-143_TSOT-6:SOT-23_Handsoldering, symbol NPN
- added R10, R11, R6, R7, R8, R9: R, Resistors_SMD:R_0603_HandSoldering, symbol R
- added SW1: SW_PUSH, igrow:SPSTSW, symbol SW_PUSH
- added U3: TL972, Housings_SOIC:SOIC-8_3.9x4.9mm_Pitch1.27mm, symbol TL972
- C1: footprint SMD_Packages:SMD-0603_c -> Capacitors_SMD:C_0603_HandSoldering
- D1: footprint SMD_Packages:SMD-0805 -> Diodes_SMD:Diode-SMC_Handsoldering
- D2, D3: footprint SMD_Packages:SMD-0805 -> LEDs:LED-0805
- Q1: footprint SMD_Packages:SOT-23 -> Housings_SOT-23_SOT-143_TSOT-6:SOT-23_Handsoldering
- R1, R2, R3, R4, R5: footprint SMD_Packages:SMD-0603_r -> Resistors_SMD:R_0603_HandSoldering
Connections:
- net GND: now also Q2.1 (E), Q3.1 (E), R7.2, SW1.2, U3.4 (V-), U3.5 (+), U3.6 (-); no longer D2.2 (K), D3.2 (K)
- net VCC: now also R10.1, R6.1, R8.1, R9.1, U3.8 (V+)
- net at U1.17 (P0.03): now also R11.1
- net at D2.1 (A): now also R8.2; no longer R1.1
- net at D3.1 (A): now also R9.2; no longer R2.1
- new net: D2.2 (K), Q2.3 (C)
- new net: D3.2 (K), Q3.3 (C)
- new net: Q2.2 (B), R1.1
- new net: Q3.2 (B), R2.1
- new net: R6.2, R7.1, U3.2 (-)
- new net: R10.2, R11.2, SW1.1
Other:
- moved on the sheet: D2, D3, R1, R2

Commit message: Post autorouting
Parts:
- BT1: footprint guan:BAT-BK912 -> igrow:CR2032_THRUHOLE
- PIEZO1: footprint Resistors_ThroughHole:Resistor_Horizontal_RM10mm -> Resistors_ThroughHole:Resistor_Vertical_RM5mm
Connections:
- net at U1.20 (P0.06): now also R2.2
- net at U1.21 (P0.07): now also R1.2
- net at U1.33 (P0.17): no longer R2.2
- net at U1.36 (P0.20): no longer R1.2
Other:
- moved on the sheet: D2, D3, D4, PIEZO1, Q1, Q2, Q3, R1, R2, R3, R4, R5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

Commit message: Flip module to other side, correct header pinout and make the module pads bigger
Parts:
- PIEZO1: footprint Resistors_ThroughHole:Resistor_Vertical_RM5mm -> Resistors_SMD:R_0805_HandSoldering
Connections:
- net VTG is gone; now on net VCC: P1.1 (P1)
- net VCC: now also BT1.1 (+)
- net at U1.1 (P0.21): no longer U2.1 (SDA)
- net at U1.17 (P0.03): no longer R11.1
- net at U1.2 (P0.22): no longer U2.6 (SCLK)
- net at U1.22 (P0.08): now also R11.1
- net at U1.35 (P0.19): now also U2.6 (SCLK)
- net at U1.36 (P0.20): now also U2.1 (SDA)
Other:
- moved on the sheet: C1, U2
Changed lines of the file:
@@
 	1100 5650 1100 5550
-Wire Wire Line
-	1100 5550 1950 5550
 Wire Wire Line
 	1800 3200 2200 3200
@@
 L SHT21 U2
 U 1 1 54D0FB67
-P 1900 2100
-F 0 "U2" H 1600 2300 60  0000 C CNN
-F 1 "SHT21" H 1600 2400 60  0000 C CNN
-F 2 "igrow:SHT21" H 1900 2100 60  0001 C CNN
-F 3 "" H 1900 2100 60  0000 C CNN
-	1    1900 2100
-	1    0    0    -1
+P 5600 1500
+F 0 "U2" H 5300 1700 60  0000 C CNN
+F 1 "SHT21" H 5300 1800 60  0000 C CNN
+F 2 "igrow:SHT21" H 5600 1500 60  0001 C CNN
+F 3 "" H 5600 1500 60  0000 C CNN
+	1    5600 1500
+	0    -1   -1   0
 $EndComp
 $Comp
 L VCC #PWR07
 U 1 1 54D0FC74
-P 1050 1850
-F 0 "#PWR07" H 1050 1700 60  0001 C CNN
-F 1 "VCC" H 1050 2000 60  0000 C CNN
-F 2 "" H 1050 1850 60  0000 C CNN
-F 3 "" H 1050 1850 60  0000 C CNN
-	1    1050 1850
+P 5500 2800
+F 0 "#PWR07" H 5500 2650 60  0001 C CNN
+F 1 "VCC" H 5500 2950 60  0000 C CNN
+F 2 "" H 5500 2800 60  0000 C CNN
+F 3 "" H 5500 2800 60  0000 C CNN
+	1    5500 2800
 	1    0    0    -1
 $EndComp
@@
 L GND #PWR08
 U 1 1 54D0FCB0
-P 1050 2550
-F 0 "#PWR08" H 1050 2300 60  0001 C CNN
-F 1 "GND" H 1050 2400 60  0000 C CNN
-F 2 "" H 1050 2550 60  0000 C CNN
-F 3 "" H 1050 2550 60  0000 C CNN
-	1    1050 2550
-	1    0    0    -1
+P 4600 1400
+F 0 "#PWR08" H 4600 1150 60  0001 C CNN
+F 1 "GND" H 4600 1250 60  0000 C CNN
+F 2 "" H 4600 1400 60  0000 C CNN
+F 3 "" H 4600 1400 60  0000 C CNN
+	1    4600 1400
+	0    1    1    0
 $EndComp
 $Comp
 L C C1
 U 1 1 54D0FCD8
-P 1050 2200
-F 0 "C1" H 1050 2300 40  0000 L CNN
-F 1 "C" H 1056 2115 40  0000 L CNN
-F 2 "Capacitors_SMD:C_0603_HandSoldering" H 1088 2050 30  0001 C CNN
-F 3 "" H 1050 2200 60  0000 C CNN
-	1    1050 2200
-	1    0    0    -1
-$EndComp
-Wire Wire Line
-	1300 2000 1050 2000
-Wire Wire Line
-	1050 2000 1050 1850
-Wire Wire Line
-	1050 2400 1050 2550
-Wire Wire Line
-	1300 2100 1250 2100
-Wire Wire Line
-	1250 2100 1250 2300
-Wire Wire Line
-	1250 2300 2200 2300
-Wire Wire Line
-	1900 2100 2050 2100
-Wire Wire Line
-	2050 2100 2050 2200
-Wire Wire Line
-	2050 2200 2200 2200
-$Comp
-L GND #PWR09
-U 1 1 54D0FFED
-P 2100 2000
-F 0 "#PWR09" H 2100 1750 60  0001 C CNN
-F 1 "GND" H 2100 1850 60  0000 C CNN
-F 2 "" H 2100 2000 60  0000 C CNN
-F 3 "" H 2100 2000 60  0000 C CNN
-	1    2100 2000
-	0    -1   -1   0
-$EndComp
-Wire Wire Line
-	2100 2000 1900 2000
+P 4800 1800
+F 0 "C1" H 4800 1900 40  0000 L CNN
+F 1 "C" H 4806 1715 40  0000 L CNN
+F 2 "Capacitors_SMD:C_0603_HandSoldering" H 4838 1650 30  0001 C CNN
+F 3 "" H 4800 1800 60  0000 C CNN
+	1    4800 1800
+	-1   0    0    1
+$EndComp
 $Comp
 L R R1
@@
 $EndComp
 $Comp
-L GND #PWR010
+L GND #PWR09
 U 1 1 54D1054F
 P 5800 5100
-F 0 "#PWR010" H 5800 4850 60  0001 C CNN
+F 0 "#PWR09" H 5800 4850 60  0001 C CNN
 F 1 "GND" H 5800 4950 60  0000 C CNN
 F 2 "" H 5800 5100 60  0000 C CNN
@@
 $EndComp
 $Comp
-L VCC #PWR011
+L VCC #PWR010
 U 1 1 54D8A9FD
 P 4300 5350
-F 0 "#PWR011" H 4300 5200 60  0001 C CNN
+F 0 "#PWR010" H 4300 5200 60  0001 C CNN
 F 1 "VCC" H 4300 5500 60  0000 C CNN
 F 2 "" H 4300 5350 60  0000 C CNN
@@
 F 0 "PIEZO1" H 4400 6450 40  0000 L CNN
 F 1 "PIEZO" H 4400 6350 40  0000 L CNN
-F 2 "Resistors_ThroughHole:Resistor_Vertical_RM5mm" H 4300 6400 60  0001 C CNN
+F 2 "Resistors_SMD:R_0805_HandSoldering" H 4300 6400 60  0001 C CNN
 F 3 "" H 4300 6400 60  0000 C CNN
 	1    4300 6400
@@
 $EndComp
 $Comp
-L GND #PWR012
+L GND #PWR011
 U 1 1 54D8ADBC
 P 4300 7450
-F 0 "#PWR012" H 4300 7200 60  0001 C CNN
+F 0 "#PWR011" H 4300 7200 60  0001 C CNN
 F 1 "GND" H 4300 7300 60  0000 C CNN
 F 2 "" H 4300 7450 60  0000 C CNN
@@
 	7050 4050 7050 4700
 $Comp
-L GND #PWR013
+L GND #PWR012
 U 1 1 54EAEC5D
 P 7050 4700
-F 0 "#PWR013" H 7050 4450 60  0001 C CNN
+F 0 "#PWR012" H 7050 4450 60  0001 C CNN
 F 1 "GND" H 7050 4550 60  0000 C CNN
 F 2 "" H 7050 4700 60  0000 C CNN
@@
 Connection ~ 7050 4250
 $Comp
-L VCC #PWR014
+L VCC #PWR013
 U 1 1 54EAEE08
 P 7450 3600
-F 0 "#PWR014" H 7450 3450 60  0001 C CNN
+F 0 "#PWR013" H 7450 3450 60  0001 C CNN
 F 1 "VCC" H 7450 3750 60  0000 C CNN
 F 2 "" H 7450 3600 60  0000 C CNN
@@
 Connection ~ 750  4500
 $Comp
-L GND #PWR015
+L GND #PWR014
 U 1 1 54EAF748
 P 750 5300
-F 0 "#PWR015" H 750 5050 60  0001 C CNN
+F 0 "#PWR014" H 750 5050 60  0001 C CNN
 F 1 "GND" H 750 5150 60  0000 C CNN
 F 2 "" H 750 5300 60  0000 C CNN
@@
 $EndComp
 $Comp
-L VCC #PWR016
+L VCC #PWR015
 U 1 1 54EAF784
 P 750 3700
-F 0 "#PWR016" H 750 3550 60  0001 C CNN
+F 0 "#PWR015" H 750 3550 60  0001 C CNN
 F 1 "VCC" H 750 3850 60  0000 C CNN
 F 2 "" H 750 3700 60  0000 C CNN
@@
 $EndComp
 $Comp
-L GND #PWR017
+L GND #PWR016
 U 1 1 54F1A792
 P 5500 4550
-F 0 "#PWR017" H 5500 4300 60  0001 C CNN
+F 0 "#PWR016" H 5500 4300 60  0001 C CNN
 F 1 "GND" H 5500 4400 60  0000 C CNN
 F 2 "" H 5500 4550 60  0000 C CNN
@@
 	5800 4500 5800 4600
 $Comp
+L VCC #PWR017
+U 1 1 54F1ABAC
+P 4600 2200
+F 0 "#PWR017" H 4600 2050 60  0001 C CNN
+F 1 "VCC" H 4600 2350 60  0000 C CNN
+F 2 "" H 4600 2200 60  0000 C CNN
+F 3 "" H 4600 2200 60  0000 C CNN
+	1    4600 2200
+	0    -1   -1   0
+$EndComp
+$Comp
 L VCC #PWR018
-U 1 1 54F1ABAC
-P 5500 2800
-F 0 "#PWR018" H 5500 2650 60  0001 C CNN
-F 1 "VCC" H 5500 2950 60  0000 C CNN
-F 2 "" H 5500 2800 60  0000 C CNN
-F 3 "" H 5500 2800 60  0000 C CNN
-	1    5500 2800
-	1    0    0    -1
-$EndComp
-$Comp
-L VCC #PWR019
 U 1 1 54F1AC2C
 P 5800 3400
-F 0 "#PWR019" H 5800 3250 60  0001 C CNN
+F 0 "#PWR018" H 5800 3250 60  0001 C CNN
 F 1 "VCC" H 5800 3550 60  0000 C CNN
 F 2 "" H 5800 3400 60  0000 C CNN
@@
 $EndComp
 $Comp
-L VCC #PWR020
+L VCC #PWR019
 U 1 1 54F1D024
 P 2400 4000
-F 0 "#PWR020" H 2400 3850 60  0001 C CNN
+F 0 "#PWR019" H 2400 3850 60  0001 C CNN
 F 1 "VCC" H 2400 4150 60  0000 C CNN
 F 2 "" H 2400 4000 60  0000 C CNN
@@
 	2400 4000 2400 4100
 $Comp
-L GND #PWR021
+L GND #PWR020
 U 1 1 54F1D139
 P 2400 5400
-F 0 "#PWR021" H 2400 5150 60  0001 C CNN
+F 0 "#PWR020" H 2400 5150 60  0001 C CNN
 F 1 "GND" H 2400 5250 60  0000 C CNN
 F 2 "" H 2400 5400 60  0000 C CNN
@@
 $EndComp
 Wire Wire Line
-	3000 4600 3000 3900
+	3000 4600 3500 4600
 Wire Wire Line
 	2400 4600 2500 4600
@@
 	3900 7100 4000 7100
 Wire Wire Line
-	4300 6900 4300 6550
-Wire Wire Line
-	4300 6250 4300 6000
+	4300 6550 4300 6900
+Wire Wire Line
+	4300 6000 4300 6250
 Wire Wire Line
 	4300 5500 4300 5350
@@
 Wire Wire Line
 	3300 4800 3300 3900
+$Comp
+L VTG #PWR021
+U 1 1 5528FD36
+P 1950 5800
+F 0 "#PWR021" H 1950 5650 60  0001 C CNN
+F 1 "VTG" H 1950 5950 60  0000 C CNN
+F 2 "" H 1950 5800 60  0000 C CNN
+F 3 "" H 1950 5800 60  0000 C CNN
+	1    1950 5800
+	0    1    1    0
+$EndComp
+Wire Wire Line
+	1900 5550 1900 5800
+Wire Wire Line
+	1900 5800 1950 5800
+Connection ~ 1900 5550
+Wire Wire Line
+	5600 1500 5600 1300
+Wire Wire Line
+	5600 1300 4200 1300
+Wire Wire Line
+	4200 1300 4200 2200
+Wire Wire Line
+	4200 2200 4100 2200
+Wire Wire Line
+	5600 2100 5600 2300
+Wire Wire Line
+	5600 2300 4100 2300
+Wire Wire Line
+	5500 1400 5500 1500
+Wire Wire Line
+	4600 1400 5500 1400
+Wire Wire Line
+	4800 1600 4800 1400
+Connection ~ 4800 1400
+Wire Wire Line
+	5500 2200 5500 2100
+Wire Wire Line
+	4600 2200 5500 2200
+Wire Wire Line
+	4800 2000 4800 2200
+Connection ~ 4800 2200
+Wire Wire Line
+	3500 4600 3500 3900
+Wire Wire Line
+	1100 5550 1950 5550
+Connection ~ 1550 5550
 $EndSCHEMATC
