File: igrow-101/igrow-101.sch (KiCad schematic (older format))
At the start: 26 parts, among them P1 CONN_02X05, Q1 NPN, Q2 NPN, Q3 NPN, SW1 SW_PUSH, U1 NRF51822-MODULE, U2 SHT21, U3 TL972

Commit message: First pass at board revision D - use direct connected IR LEDs for sensing
Parts:
- removed R6: R, Resistors_SMD:R_0603_HandSoldering, symbol R
- removed U3: TL972, Housings_SOIC:SOIC-8_3.9x4.9mm_Pitch1.27mm, symbol TL972
- added D3, D4, D5: LED, LEDs:LED-5MM, symbol LED
- added P2, P3, P4, P5: CONN_01X01, igrow:MountingHole_M3, symbol CONN_01X01
- added R5, R8: R, Resistors_SMD:R_0603_HandSoldering, symbol R
- added W1: TEST_1P, Measurement_Points:Measurement_Point_Round-TH_Big, symbol TEST_1P
- C1: symbol C -> C-RESCUE-igrow-101
- D2: renamed from D4; symbol ZENER -> ZENER-RESCUE-igrow-101
- D6: renamed from D2; symbol LED -> LED-RESCUE-igrow-101
- D7: renamed from D3; symbol LED -> LED-RESCUE-igrow-101
- Q1, Q2, Q3: footprint Housings_SOT-23_SOT-143_TSOT-6:SOT-23_Handsoldering -> igrow:SOT-23_Handsoldering_EBC
- R1: renamed from R10; symbol R -> R-RESCUE-igrow-101
- R10: renamed from R2; symbol R -> R-RESCUE-igrow-101
- R11: renamed from R8; symbol R -> R-RESCUE-igrow-101
- R12: renamed from R9; symbol R -> R-RESCUE-igrow-101
- R2: renamed from R11; symbol R -> R-RESCUE-igrow-101
- R3, R4: symbol R -> R-RESCUE-igrow-101
- R6: renamed from R5; symbol R -> R-RESCUE-igrow-101
- R9: renamed from R1; symbol R -> R-RESCUE-igrow-101
Connections:
- wire segments 69 -> 78
Other:
- moved on the sheet: D6, D7, P1, Q2, Q3, R10, R11, R12, R9

Commit message: Revision D as sent to dirtypcbs for fab
Parts:
- D6, D7: footprint LEDs:LED-0805 -> LEDs:LED_0805
Changed lines of the file:
@@
 Sheet 1 1
 Title "iGrow Pebble 101"
-Date "Saturday, 25 April 2015"
-Rev "C"
+Date "2016-06-09"
+Rev "D"
 Comp "Argusat Limited"
 Comment1 ""
@@
 F 0 "D6" H 7400 3800 50  0000 C CNN
 F 1 "LED" H 7400 3600 50  0000 C CNN
-F 2 "LEDs:LED-0805" H 7400 3700 60  0001 C CNN
+F 2 "LEDs:LED_0805" H 7400 3700 60  0001 C CNN
 F 3 "" H 7400 3700 60  0000 C CNN
 	1    7400 3700
@@
 F 0 "D7" H 7700 4400 50  0000 C CNN
 F 1 "LED" H 7700 4200 50  0000 C CNN
-F 2 "LEDs:LED-0805" H 7700 4300 60  0001 C CNN
+F 2 "LEDs:LED_0805" H 7700 4300 60  0001 C CNN
 F 3 "" H 7700 4300 60  0000 C CNN
 	1    7700 4300

Commit message: Fix diode calibrator script.  Add updated LED model.  Add calculated schematic values.  Add Matlab/octave scripts for plotting simulation output.
Parts:
- C1: value C -> 100nF
- R1, R10, R9: value R -> 10kR
- R11, R12: value R -> 620R
- R2: value R -> 150R
- R5, R7, R8: value R -> 220R
Changed lines of the file:
@@
 F 1 "LED" H 7400 3600 50  0000 C CNN
 F 2 "LEDs:LED_0805" H 7400 3700 60  0001 C CNN
-F 3 "" H 7400 3700 60  0000 C CNN
+F 3 "osram_LGT67K" H 7400 3700 60  0000 C CNN
 	1    7400 3700
 	0    1    1    0
@@
 P 4800 1800
 F 0 "C1" H 4800 1900 40  0000 L CNN
-F 1 "C" H 4806 1715 40  0000 L CNN
+F 1 "100nF" H 4806 1715 40  0000 L CNN
 F 2 "Capacitors_SMD:C_0603_HandSoldering" H 4838 1650 30  0001 C CNN
 F 3 "" H 4800 1800 60  0000 C CNN
@@
 P 6550 4200
 F 0 "R9" V 6630 4200 40  0000 C CNN
-F 1 "R" V 6557 4201 40  0000 C CNN
+F 1 "10kR" V 6557 4201 40  0000 C CNN
 F 2 "Resistors_SMD:R_0603_HandSoldering" V 6480 4200 30  0001 C CNN
 F 3 "" H 6550 4200 30  0000 C CNN
@@
 P 6650 4800
 F 0 "R10" V 6730 4800 40  0000 C CNN
-F 1 "R" V 6657 4801 40  0000 C CNN
+F 1 "10kR" V 6657 4801 40  0000 C CNN
 F 2 "Resistors_SMD:R_0603_HandSoldering" V 6580 4800 30  0001 C CNN
 F 3 "" H 6650 4800 30  0000 C CNN
@@
 P 7400 3150
 F 0 "R11" V 7480 3150 40  0000 C CNN
-F 1 "R" V 7407 3151 40  0000 C CNN
+F 1 "620R" V 7407 3151 40  0000 C CNN
 F 2 "Resistors_SMD:R_0603_HandSoldering" V 7330 3150 30  0001 C CNN
 F 3 "" H 7400 3150 30  0000 C CNN
@@
 P 7700 3750
 F 0 "R12" V 7780 3750 40  0000 C CNN
-F 1 "R" V 7707 3751 40  0000 C CNN
+F 1 "620R" V 7707 3751 40  0000 C CNN
 F 2 "Resistors_SMD:R_0603_HandSoldering" V 7630 3750 30  0001 C CNN
 F 3 "" H 7700 3750 30  0000 C CNN
@@
 P 2400 4350
 F 0 "R1" V 2480 4350 40  0000 C CNN
-F 1 "R" V 2407 4351 40  0000 C CNN
+F 1 "10kR" V 2407 4351 40  0000 C CNN
 F 2 "Resistors_SMD:R_0603_HandSoldering" V 2330 4350 30  0001 C CNN
 F 3 "" H 2400 4350 30  0000 C CNN
@@
 P 2750 4600
 F 0 "R2" V 2830 4600 40  0000 C CNN
-F 1 "R" V 2757 4601 40  0000 C CNN
+F 1 "150R" V 2757 4601 40  0000 C CNN
 F 2 "Resistors_SMD:R_0603_HandSoldering" V 2680 4600 30  0001 C CNN
 F 3 "" H 2750 4600 30  0000 C CNN
@@
 P 4400 3250
 F 0 "R5" V 4480 3250 50  0000 C CNN
-F 1 "R" V 4400 3250 50  0000 C CNN
+F 1 "220R" V 4400 3250 50  0000 C CNN
 F 2 "Resistors_SMD:R_0603_HandSoldering" V 4330 3250 50  0001 C CNN
 F 3 "" H 4400 3250 50  0000 C CNN
@@
 P 4800 3250
 F 0 "R7" V 4880 3250 50  0000 C CNN
-F 1 "R" V 4800 3250 50  0000 C CNN
+F 1 "220R" V 4800 3250 50  0000 C CNN
 F 2 "Resistors_SMD:R_0603_HandSoldering" V 4730 3250 50  0001 C CNN
 F 3 "" H 4800 3250 50  0000 C CNN
@@
 P 5100 3250
 F 0 "R8" V 5180 3250 50  0000 C CNN
-F 1 "R" V 5100 3250 50  0000 C CNN
+F 1 "220R" V 5100 3250 50  0000 C CNN
 F 2 "Resistors_SMD:R_0603_HandSoldering" V 5030 3250 50  0001 C CNN
 F 3 "" H 5100 3250 50  0000 C CNN

Commit message: Correct sizing for module, button cell holder through-holes and enlarge SHT21 pads to allow hand soldering if required.
Parts:
- U2: footprint igrow:SHT21 -> igrow:SHT21_HandSoldering
Changed lines of the file:
@@
 F 0 "U2" H 5300 1700 60  0000 C CNN
 F 1 "SHT21" H 5300 1800 60  0000 C CNN
-F 2 "igrow:SHT21" H 5600 1500 60  0001 C CNN
+F 2 "igrow:SHT21_HandSoldering" H 5600 1500 60  0001 C CNN
 F 3 "" H 5600 1500 60  0000 C CNN
 	1    5600 1500
