File: igrow-101/_autosave-igrow-101.kicad_pcb (KiCad board)
At the start: 2 copper layers, 49.8 x 39.5 mm, 34 parts, among them P1 CONN_02X05, P2 CONN_01X01, P3 CONN_01X01, P4 CONN_01X01, P5 CONN_01X01, Q1 NPN, Q2 NPN, Q3 NPN, SW1 SW_PUSH, U1 NRF51822-MODULE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

Commit message: Hardware revision F
Other:
- board text added: "iGrow 101 (c) 2016 Argusat Limited"
Changed lines of the file:
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@@
-(kicad_pcb (version 4) (host pcbnew 4.0.3+e1-6302~38~ubuntu16.04.1-stable)
+(kicad_pcb (version 4) (host pcbnew 4.0.4+e1-6308~48~ubuntu16.04.1-stable)
   (general
     (links 57)
     (no_connects 0)
-    (area 131.242999 93.142999 181.177001 132.790001)
+    (area 129.146 91.554 182.887334 133.669)
     (thickness 1.6)
-    (drawings 9)
+    (drawings 10)
     (tracks 245)
     (zones 0)
@@
     (visible_elements FFFFFF7F)
     (pcbplotparams
-      (layerselection 0x010fc_80000001)
-      (usegerberextensions true)
-      (usegerberattributes true)
+      (layerselection 0x0000c_00000000)
+      (usegerberextensions false)
       (excludeedgelayer true)
       (linewidth 0.100000)
@@
       (padsonsilk false)
       (subtractmaskfromsilk false)
-      (outputformat 1)
+      (outputformat 5)
       (mirror false)
       (drillshape 0)
       (scaleselection 1)
-      (outputdirectory fab))
+      (outputdirectory svg))
   )
   (net 0 "")
@@
     (tags "capacitor 0603")
     (attr smd)
-    (fp_text reference C1 (at 0 -1.27 90) (layer F.SilkS)
+    (fp_text reference C1 (at 2.675 -0.475 180) (layer F.SilkS)
       (effects (font (size 1 1) (thickness 0.15)))
     )
@@
     (tags "resistor 0603")
     (attr smd)
-    (fp_text reference R1 (at -2.794 0 270) (layer F.SilkS)
+    (fp_text reference R1 (at 0 1.66 270) (layer F.SilkS)
       (effects (font (size 1 1) (thickness 0.15)))
     )
@@
     (tags "resistor 0603")
     (attr smd)
-    (fp_text reference R2 (at -2.921 0) (layer F.SilkS)
+    (fp_text reference R2 (at 0.11 1.575) (layer F.SilkS)
       (effects (font (size 1 1) (thickness 0.15)))
     )
@@
     (tags "resistor 0603")
     (attr smd)
-    (fp_text reference R3 (at -2.794 0) (layer F.SilkS)
+    (fp_text reference R3 (at -0.015 1.575) (layer F.SilkS)
       (effects (font (size 1 1) (thickness 0.15)))
     )
@@
     (tags "resistor 0603")
     (attr smd)
-    (fp_text reference R4 (at -0.254 -1.27 270) (layer F.SilkS)
+    (fp_text reference R4 (at -0.11 -1.89 270) (layer F.SilkS)
       (effects (font (size 1 1) (thickness 0.15)))
     )
@@
     (tags "resistor 0603")
     (attr smd)
-    (fp_text reference R5 (at -0.254 -1.27 90) (layer F.SilkS)
+    (fp_text reference R5 (at 0.125 1.815 90) (layer F.SilkS)
       (effects (font (size 1 1) (thickness 0.15)))
     )
@@
     (tags "resistor 0603")
     (attr smd)
-    (fp_text reference R6 (at -3.302 0) (layer F.SilkS)
+    (fp_text reference R6 (at -0.125 -1.685) (layer F.SilkS)
       (effects (font (size 1 1) (thickness 0.15)))
     )
@@
     (tags "resistor 0603")
     (attr smd)
-    (fp_text reference R8 (at 0.127 -1.397 90) (layer F.SilkS)
+    (fp_text reference R8 (at 2.675 -0.435 180) (layer F.SilkS)
       (effects (font (size 1 1) (thickness 0.15)))
     )
@@
     (tags "resistor 0603")
     (attr smd)
-    (fp_text reference R10 (at 3.175 0) (layer F.SilkS)
+    (fp_text reference R10 (at 0.035 1.425) (layer F.SilkS)
       (effects (font (size 1 1) (thickness 0.15)))
     )
@@
     (tags "resistor 0603")
     (attr smd)
-    (fp_text reference R11 (at 3.048 0) (layer F.SilkS)
+    (fp_text reference R11 (at 0.11 1.465) (layer F.SilkS)
       (effects (font (size 1 1) (thickness 0.15)))
     )
@@
   (module igrow:SPSTSW (layer F.Cu)
     (at 162.56 127 180)
-    (fp_text reference SW1 (at 2.54 2.54 180) (layer F.SilkS)
+    (fp_text reference SW1 (at 5.31 6.75 360) (layer F.SilkS)
       (effects (font (size 1.5 1.5) (thickness 0.15)))
     )
@@
     (tags "resistor 0805")
     (attr smd)
-    (fp_text reference PIEZO1 (at -0.254 -1.524 270) (layer F.SilkS)
+    (fp_text reference PIEZO1 (at 0.116 -2.054 270) (layer F.SilkS)
       (effects (font (size 1 1) (thickness 0.15)))
     )
@@
   (module igrow:harwin_m50-3600542 (layer F.Cu)
     (at 153.67 107.95 180)
-    (fp_text reference P1 (at 2.54 6.985 180) (layer F.SilkS)
+    (fp_text reference P1 (at 1.67 -2.05 180) (layer F.SilkS)
       (effects (font (size 1.5 1.5) (thickness 0.15)))
     )
@@
     (descr "LED 5mm round vertical")
     (tags "LED 5mm round vertical")
-    (fp_text reference D3 (at 1.524 -4.064 180) (layer B.SilkS)
+    (fp_text reference D3 (at -1.875 2.45 180) (layer B.SilkS)
       (effects (font (size 1 1) (thickness 0.15)) (justify mirror))
     )
@@
     (descr "LED 5mm round vertical")
     (tags "LED 5mm round vertical")
-    (fp_text reference D4 (at 1.524 -4.064 180) (layer B.SilkS)
+    (fp_text reference D4 (at 4.875 2.485 180) (layer B.SilkS)
       (effects (font (size 1 1) (thickness 0.15)) (justify mirror))
     )
@@
     (descr "LED 5mm round vertical")
     (tags "LED 5mm round vertical")
-    (fp_text reference D5 (at 1.524 -4.064 180) (layer B.SilkS)
+    (fp_text reference D5 (at 4.875 2.27 180) (layer B.SilkS)
       (effects (font (size 1 1) (thickness 0.15)) (justify mirror))
     )
@@
     (tags "resistor 0603")
     (attr smd)
-    (fp_text reference R12 (at 0 -1.9 270) (layer F.SilkS)
+    (fp_text reference R12 (at -2.84 -0.18 360) (layer F.SilkS)
       (effects (font (size 1 1) (thickness 0.15)))
     )
@@
   (module igrow:MountingHole_M3 (layer F.Cu)
     (at 134.62 96.52)
-    (fp_text reference P2 (at 0 0.5) (layer F.SilkS)
+    (fp_text reference P2 (at -2.12 2.73) (layer F.SilkS)
       (effects (font (size 1 1) (thickness 0.15)))
     )
@@
   (module igrow:MountingHole_M3 (layer F.Cu)
     (at 134.62 129.54)
-    (fp_text reference P3 (at 0 0.5) (layer F.SilkS)
+    (fp_text reference P3 (at -1.87 -2.79) (layer F.SilkS)
       (effects (font (size 1 1) (thickness 0.15)))
     )
@@
   (module igrow:MountingHole_M3 (layer F.Cu)
     (at 177.8 129.54)
-    (fp_text reference P4 (at 0 0.5) (layer F.SilkS)
+    (fp_text reference P4 (at -2.3 -2.54) (layer F.SilkS)
       (effects (font (size 1 1) (thickness 0.15)))
     )
@@
   (module igrow:MountingHole_M3 (layer F.Cu)
     (at 177.8 96.52)
-    (fp_text reference P5 (at 0 0.5) (layer F.SilkS)
+    (fp_text reference P5 (at 1.45 3.23) (layer F.SilkS)
       (effects (font (size 1 1) (thickness 0.15)))
     )
@@
     (tags SOT-23)
     (attr smd)
-    (fp_text reference Q1 (at 0 -3.81) (layer F.SilkS)
+    (fp_text reference Q1 (at 0.14 3.54) (layer F.SilkS)
       (effects (font (size 1 1) (thickness 0.15)))
     )
@@
     (tags SOT-23)
     (attr smd)
-    (fp_text reference Q2 (at 0 -3.81) (layer F.SilkS)
+    (fp_text reference Q2 (at -0.02 3.445) (layer F.SilkS)
       (effects (font (size 1 1) (thickness 0.15)))
     )
@@
     (tags SOT-23)
     (attr smd)
-    (fp_text reference Q3 (at 0 -3.81 270) (layer F.SilkS)
+    (fp_text reference Q3 (at -2.425 0.905 540) (layer F.SilkS)
       (effects (font (size 1 1) (thickness 0.15)))
     )
@@
     (tags "Mesurement Point Round Trough Hole 3mm 1.5mm")
     (attr virtual)
-    (fp_text reference W1 (at 0 -3) (layer F.SilkS)
+    (fp_text reference W1 (at -1.22 -2.29) (layer F.SilkS)
       (effects (font (size 1 1) (thickness 0.15)))
     )
@@
       (net 1 GND))
   )
+  (gr_text "iGrow 101\n(c) 2016\nArgusat Limited" (at 150 101.25) (layer B.SilkS)
+    (effects (font (size 0.75 0.75) (thickness 0.1875)) (justify mirror))
+  )
   (target plus (at 134.62 129.54) (size 5) (width 0.15) (layer Edge.Cuts))
